File: esp8266.kicad_sch (KiCad schematic)
At the start: 47 parts, among them J1 Conn_01x08, J2 Conn_01x08, Q1 AO3401A, U10 RST, U11 W25Q128JVSIQTR, U13 CH340C, U2 ESP8266EX, U3 AP2112K-3_3TRG1, U4 HDC1080DMBR, U5 MCP73831T-2ACI_OT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

Commit message: Rework layout to retain power and ground plane continuity.
Add one more decoupling capacitor to CH340.

The ground plane now has islands of shorter traces. The 3.3V plane has been carefully adjusted to provide reasonable impedances to all loads.
Parts:
- added C11, C14, C15: 100n, jlc_footprints:C0603, symbol Device:C
- C10, C8: symbol jlc_symbols:CC0603KRX7R9BB104 -> Device:C
- R8, R9: footprint Resistor_SMD:R_0603_1608Metric_Pad0.98x0.95mm_HandSolder -> jlc_footprints:R0603
- U13: footprint jlc_footprints:SOP-16_L10.0-W3.9-P1.27-LS6.0-BL -> Package_SO:SOIC-16_3.9x9.9mm_P1.27mm
Connections:
- net +3V3: now also U13.10 (~{DSR}), U13.9 (~{CTS}), C11.2, C14.2, C15.2
- net DTR: now also U13.11 (~{RI}), U13.12 (~{DCD})
- net GND: now also C11.1, C14.1, C15.1
- no-connect marks 18 -> 15
